Commit message: right_shoulder_x fixed

File: urdf/gingerurdf.urdf (robot description, URDF)
Before this commit: robot gingerurdf, 50 links, 49 joints
Joints:
- joint RIght_Shoulder__X: axis 0 0 1 -> 1 0 0

Commit message: Actually fix right shoulder

File: urdf/gingerurdf.urdf (robot description, URDF)
Before this commit: robot gingerurdf, 50 links, 49 joints
Links:
- removed link RIght_Shoulder_X_Link
- added link Right_Shoulder_X_Link, mass 0.268082573106329; collision mesh filename=package://gingerurdf/meshes/Right_Shoulder_X_Link.STL; visual mesh filename=package://gingerurdf/meshes/Right_Shoulder_X_Link.STL
Joints:
- removed joint RIght_Shoulder__X
- added joint Right_Shoulder_X: type continuous, parent Back_Y_Link, child Right_Shoulder_X_Link, origin xyz=-0.167642819137822 0.257434208389716 -0.0153204612848374 rpy=5.79452944416604E-17 -1.59192802633449E-16 -0.349087221077984, axis 1 0 0
- joint Right_Shoulder_Y: parent RIght_Shoulder_X_Link -> Right_Shoulder_X_Link

Commit message: update continue joint -> revolute joint, also add limit
Change-Id: Ic3c924edc31709988516400d788746822d9bc1a5

File: urdf/gingerurdf.urdf (robot description, URDF)
Before this commit: robot gingerurdf, 50 links, 49 joints
Joints:
- joint Back_X: limit (none) -> lower=-0.78190750489346 upper=0.991347015132779 effort=30 velocity=1.0; type continuous -> revolute
- joint Back_Y: limit (none) -> lower=-0.720820981073658 upper=0.720820981073658 effort=30 velocity=1.0; type continuous -> revolute
- joint Back_Z: limit (none) -> lower=-1.69488923661169 upper=1.69488923661169 effort=30 velocity=1.0; type continuous -> revolute
- joint Head_Y: limit (none) -> lower=-0.441917366604964 upper=0.441917366604964 effort=30 velocity=1.0; type continuous -> revolute
- joint Knee: limit (none) -> lower=-0.62779493194236 upper=0.539830337641846 effort=30 velocity=1.0; type continuous -> revolute
- joint Left_1_1: limit (none) -> lower=0 upper=1.25663706143592 effort=30 velocity=1.0; type continuous -> revolute
- joint Left_1_2: limit (none) -> lower=0 upper=1.25663706143592 effort=30 velocity=1.0; type continuous -> revolute
- joint Left_2_1: limit (none) -> lower=0 upper=1.25663706143592 effort=30 velocity=1.0; type continuous -> revolute
- joint Left_2_2: limit (none) -> lower=0 upper=1.25663706143592 effort=30 velocity=1.0; type continuous -> revolute
- joint Left_2_3: limit (none) -> lower=0 upper=1.25663706143592 effort=30 velocity=1.0; type continuous -> revolute
- joint Left_3_1: limit (none) -> lower=0 upper=1.25663706143592 effort=30 velocity=1.0; type continuous -> revolute
- joint Left_3_2: limit (none) -> lower=0 upper=1.25663706143592 effort=30 velocity=1.0; type continuous -> revolute
- joint Left_3_3: limit (none) -> lower=0 upper=1.25663706143592 effort=30 velocity=1.0; type continuous -> revolute
- joint Left_4_1: limit (none) -> lower=0 upper=1.25663706143592 effort=30 velocity=1.0; type continuous -> revolute
- joint Left_4_2: limit (none) -> lower=0 upper=1.25663706143592 effort=30 velocity=1.0; type continuous -> revolute
- joint Left_4_3: limit (none) -> lower=0 upper=1.25663706143592 effort=30 velocity=1.0; type continuous -> revolute
- joint Left_5_1: limit (none) -> lower=0 upper=1.25663706143592 effort=30 velocity=1.0; type continuous -> revolute
- joint Left_5_2: limit (none) -> lower=0 upper=1.25663706143592 effort=30 velocity=1.0; type continuous -> revolute
- joint Left_5_3: limit (none) -> lower=0 upper=1.25663706143592 effort=30 velocity=1.0; type continuous -> revolute
- joint Left_Elbow_X: limit (none) -> lower=-1.61512768979555 upper=0.6770132168486 effort=30 velocity=1.0; type continuous -> revolute
- joint Left_Elbow_Z: limit (none) -> lower=-1.5707963267949 upper=1.5707963267949 effort=30 velocity=1.0; type continuous -> revolute
- joint Left_Shoulder_X: limit (none) -> lower=-3.14159265358979 upper=3.14159265358979 effort=30 velocity=1.0; type continuous -> revolute
- joint Left_Shoulder_Y: limit (none) -> lower=-0.0162315620435473 upper=1.73084301920278 effort=30 velocity=1.0; type continuous -> revolute
- joint Left_Wrist_X: limit (none) -> lower=-0.738274273593601 upper=0.738274273593601 effort=30 velocity=1.0; type continuous -> revolute
- joint Left_Wrist_Y: limit (none) -> lower=-0.523598775598299 upper=0.523598775598299 effort=30 velocity=1.0; type continuous -> revolute
- joint Left_Wrist_Z: limit (none) -> lower=-1.5707963267949 upper=1.5707963267949 effort=30 velocity=1.0; type continuous -> revolute
- joint Neck_X: limit (none) -> lower=-0.803898653468588 upper=0.417133691226645 effort=30 velocity=1.0; type continuous -> revolute
- joint Neck_Z: limit (none) -> lower=-1.5707963267949 upper=1.5707963267949 effort=30 velocity=1.0; type continuous -> revolute
- joint Right_1_1: limit (none) -> lower=0 upper=1.25663706143592 effort=30 velocity=1.0; type continuous -> revolute
- joint Right_1_2: limit (none) -> lower=0 upper=1.25663706143592 effort=30 velocity=1.0; type continuous -> revolute
- joint Right_2_1: limit (none) -> lower=0 upper=1.25663706143592 effort=30 velocity=1.0; type continuous -> revolute
- joint Right_2_2: limit (none) -> lower=0 upper=1.25663706143592 effort=30 velocity=1.0; type continuous -> revolute
- joint Right_2_3: limit (none) -> lower=0 upper=1.25663706143592 effort=30 velocity=1.0; type continuous -> revolute
- joint Right_3_1: limit (none) -> lower=0 upper=1.25663706143592 effort=30 velocity=1.0; type continuous -> revolute
- joint Right_3_2: limit (none) -> lower=0 upper=1.25663706143592 effort=30 velocity=1.0; type continuous -> revolute
- joint Right_3_3: limit (none) -> lower=0 upper=1.25663706143592 effort=30 velocity=1.0; type continuous -> revolute
- joint Right_4_1: limit (none) -> lower=0 upper=1.25663706143592 effort=30 velocity=1.0; type continuous -> revolute
- joint Right_4_2: limit (none) -> lower=0 upper=1.25663706143592 effort=30 velocity=1.0; type continuous -> revolute
- joint Right_4_3: limit (none) -> lower=0 upper=1.25663706143592 effort=30 velocity=1.0; type continuous -> revolute
- joint Right_5_1: limit (none) -> lower=0 upper=1.25663706143592 effort=30 velocity=1.0; type continuous -> revolute
- joint Right_5_2: limit (none) -> lower=0 upper=1.25663706143592 effort=30 velocity=1.0; type continuous -> revolute
- joint Right_5_3: limit (none) -> lower=0 upper=1.25663706143592 effort=30 velocity=1.0; type continuous -> revolute
- joint Right_Elbow_X: limit (none) -> lower=-1.61512768979555 upper=0.6770132168486 effort=30 velocity=1.0; type continuous -> revolute
- joint Right_Elbow_Z: limit (none) -> lower=-1.5707963267949 upper=1.5707963267949 effort=30 velocity=1.0; type continuous -> revolute
- joint Right_Shoulder_X: limit (none) -> lower=-3.14159265358979 upper=3.14159265358979 effort=30 velocity=1.0; type continuous -> revolute
- joint Right_Shoulder_Y: limit (none) -> lower=-1.73084301920278 upper=0.0162315620435473 effort=30 velocity=1.0; type continuous -> revolute
- joint Right_Wrist_X: limit (none) -> lower=-0.738274273593601 upper=0.738274273593601 effort=30 velocity=1.0; type continuous -> revolute
- joint Right_Wrist_Y: limit (none) -> lower=-0.523598775598299 upper=0.523598775598299 effort=30 velocity=1.0; type continuous -> revolute
- joint Right_Wrist_Z: limit (none) -> lower=-1.5707963267949 upper=1.5707963267949 effort=30 velocity=1.0; type continuous -> revolute

Commit message: update coordinate
Change-Id: I6ea5d02b103e181d6ba1cc94f64094af85c88953

File: urdf/gingerurdf.urdf (robot description, URDF)
Before this commit: robot gingerurdf, 50 links, 49 joints
Links:
- link base_link: mass None -> 36.8100641165154
Joints:
- joint Back_X: axis 1 0 0 -> 0 0 1; origin xyz=0 0 0 rpy=0 0 0 -> xyz=0 0 0 rpy=0 -1.5707963267949 1.5707963267949
- joint Back_Y: origin xyz=0 0.104999999999997 0 rpy=0 0 0 -> xyz=0.104999999999997 0 0 rpy=0 -1.5707963267949 1.5707963267949
- joint Back_Z: axis 0 1 0 -> 0 0 1; origin xyz=-0.0258402466955493 0.459273873742399 0 rpy=3.14159265358979 0.857307531298485 -3.0853883378301 -> xyz=0.0258402466955493 0.459273873742399 0.015 rpy=-1.5707963267949 0 0
- joint Head_Y: origin xyz=0 0.0609748006263349 0.000155084351385615 rpy=0 0 0 -> xyz=0.0609748006263349 0 0 rpy=0 1.5707963267949 -1.5707963267949
- joint Knee: axis -0.653442120633779 -0.0367649880485583 -0.756083150609388 -> 0 0 1; origin xyz=0 -0.163753578960292 0.422732937784996 rpy=1.5707963267949 0.0562043157596906 -2.28428512229131 -> xyz=0 -0.163753578960292 0.422732937784996 rpy=1.5707963267949 0 1.5707963267949
- joint Left_Elbow_X: axis 1 0 0 -> 0 0 1; origin xyz=0 0 0 rpy=0 0 0 -> xyz=0 0 0 rpy=1.5707963267949 0 0
- joint Left_Elbow_Z: axis 0 -1 0 -> 0 0 1; origin xyz=0.030674616894137 -0.227909089065574 0 rpy=3.14159265358979 0 -2.79254817387005 -> xyz=0.0491247882 0.2246558260 0 rpy=0 1.5707963267949 1.5707963267949
- joint Left_Shoulder_X: axis -1 0 0 -> 0 0 -1; origin xyz=0.167642819139667 0.257434208387602 -0.0153204612848375 rpy=3.14159265358979 0 -2.79254817387005 -> xyz=0.167642819139667 -0.257434208387602 0.0153204612848375 rpy=1.5707963267949 0 -1.919840807
- joint Left_Shoulder_Y: origin xyz=0 0 0 rpy=0 0 0 -> xyz=0 0 0 rpy=-1.5707963267949 1.919840807 0
- joint Left_Wrist_X: axis 1 0 0 -> 0 0 1; origin xyz=0 0 0 rpy=0 0 0 -> xyz=0 0 0 rpy=1.5707963267949 -1.5707963267949 0
- joint Left_Wrist_Y: origin xyz=0 0 0 rpy=0 0 0 -> xyz=0 0 0 rpy=0 -1.5707963267949 1.5707963267949
- joint Left_Wrist_Z: axis 0 -1 0 -> 0 0 1; origin xyz=-0.000196700073873679 -0.209557803287771 0.000545980735265489 rpy=0 0 0 -> xyz=0 0.209557803287771 0 rpy=-1.5707963267949 0 0
- joint Neck_X: axis 1 0 0 -> 0 0 1; origin xyz=0 0 0 rpy=0 0 0 -> xyz=0 0 0 rpy=0 -1.5707963267949 -1.5707963267949
- joint Neck_Z: axis 0 1 0 -> 0 0 1; origin xyz=0 0.37820748993899 0.00368296133076892 rpy=0 0 0 -> xyz=0 -0.37820748993899 0 rpy=0 1.5707963267949 -1.5707963267949
- joint Right_Elbow_X: axis 1 0 0 -> 0 0 1; origin xyz=0 0 0 rpy=0 0 0 -> xyz=0 0 0 rpy=1.5707963267949 0 0
- joint Right_Elbow_Z: axis 0 -1 0 -> 0 0 1; origin xyz=0.0308685949686061 -0.227838852240102 0 rpy=1.15825157085799E-32 1.69410759865549E-16 0.349087221077984 -> xyz=-0.0491247882 0.2246558260 0 rpy=0 1.5707963267949 1.5707963267949
- joint Right_Shoulder_X: axis 1 0 0 -> 0 0 1; origin xyz=-0.167642819137822 0.257434208389716 -0.0153204612848374 rpy=5.79452944416604E-17 -1.59192802633449E-16 -0.349087221077984 -> xyz=-0.167642819137822 -0.257434208389716 0.0153204612848374 rpy=-1.5707963267949 0 -1.221709106
- joint Right_Shoulder_Y: origin xyz=0 0 0 rpy=0 0 9.22447382158831E-33 -> xyz=0 0 0 rpy=1.5707963267949 -1.221709106 0
- joint Right_Wrist_X: axis 1 0 0 -> 0 0 1; origin xyz=0 0 0 rpy=0 0 0 -> xyz=0 0 0 rpy=0 -1.5707963267949 1.5707963267949
- joint Right_Wrist_Y: origin xyz=0 0 0 rpy=0 0 0 -> xyz=0 0 0 rpy=0 -1.5707963267949 1.5707963267949
- joint Right_Wrist_Z: axis 0 -1 0 -> 0 0 1; origin xyz=0 -0.209559555159009 0.000544952004672944 rpy=0 0 0 -> xyz=0 0.209559555159009 0 rpy=-1.5707963267949 0 0

Commit message: update coordinate
Change-Id: I0114aef9f3fd61ac5050c9f3f06315f11e23d55d

File: urdf/gingerurdf.urdf (robot description, URDF)
Before this commit: robot gingerurdf, 50 links, 49 joints
Joints:
- joint Back_X: axis 1 0 0 -> 0 0 1; origin xyz=0 0 0 rpy=0 0 0 -> xyz=0 0 0 rpy=0 -1.5707963267949 1.5707963267949
- joint Back_Y: origin xyz=0 0.104999999999997 0 rpy=0 0 0 -> xyz=0.104999999999997 0 0 rpy=0 -1.5707963267949 1.5707963267949
- joint Back_Z: axis 0 1 0 -> 0 0 1; origin xyz=-0.0258402466955493 0.459273873742399 0 rpy=3.14159265358979 0.857307531298485 -3.0853883378301 -> xyz=0.0258402466955493 0.459273873742399 0.015 rpy=-1.5707963267949 0 0
- joint Head_Y: origin xyz=0 0.0609748006263349 0.000155084351385615 rpy=0 0 0 -> xyz=0.0609748006263349 0 0 rpy=0 1.5707963267949 -1.5707963267949
- joint Knee: axis -0.653442120633779 -0.0367649880485583 -0.756083150609388 -> 0 0 1; origin xyz=0 -0.163753578960292 0.422732937784996 rpy=1.5707963267949 0.0562043157596906 -2.28428512229131 -> xyz=0 -0.163753578960292 0.422732937784996 rpy=1.5707963267949 0 1.5707963267949
- joint Left_Elbow_X: axis 1 0 0 -> 0 0 1; origin xyz=0 0 0 rpy=0 0 0 -> xyz=0 0 0 rpy=1.5707963267949 0 0
- joint Left_Elbow_Z: axis 0 -1 0 -> 0 0 1; origin xyz=0.030674616894137 -0.227909089065574 0 rpy=3.14159265358979 0 -2.79254817387005 -> xyz=0.0491247882 0.2246558260 0 rpy=0 1.5707963267949 1.5707963267949
- joint Left_Shoulder_X: axis -1 0 0 -> 0 0 -1; origin xyz=0.167642819139667 0.257434208387602 -0.0153204612848375 rpy=3.14159265358979 0 -2.79254817387005 -> xyz=0.167642819139667 -0.257434208387602 0.0153204612848375 rpy=1.5707963267949 0 -1.919840807
- joint Left_Shoulder_Y: origin xyz=0 0 0 rpy=0 0 0 -> xyz=0 0 0 rpy=-1.5707963267949 1.919840807 0
- joint Left_Wrist_X: axis 1 0 0 -> 0 0 1; origin xyz=0 0 0 rpy=0 0 0 -> xyz=0 0 0 rpy=1.5707963267949 -1.5707963267949 0
- joint Left_Wrist_Y: origin xyz=0 0 0 rpy=0 0 0 -> xyz=0 0 0 rpy=0 -1.5707963267949 1.5707963267949
- joint Left_Wrist_Z: axis 0 -1 0 -> 0 0 1; origin xyz=-0.000196700073873679 -0.209557803287771 0.000545980735265489 rpy=0 0 0 -> xyz=0 0.209557803287771 0 rpy=-1.5707963267949 0 0
- joint Neck_X: axis 1 0 0 -> 0 0 1; origin xyz=0 0 0 rpy=0 0 0 -> xyz=0 0 0 rpy=0 -1.5707963267949 -1.5707963267949
- joint Neck_Z: axis 0 1 0 -> 0 0 1; origin xyz=0 0.37820748993899 0.00368296133076892 rpy=0 0 0 -> xyz=0 -0.37820748993899 0 rpy=0 1.5707963267949 -1.5707963267949
- joint Right_Elbow_X: axis 1 0 0 -> 0 0 1; origin xyz=0 0 0 rpy=0 0 0 -> xyz=0 0 0 rpy=1.5707963267949 0 0
- joint Right_Elbow_Z: axis 0 -1 0 -> 0 0 1; origin xyz=0.0308685949686061 -0.227838852240102 0 rpy=1.15825157085799E-32 1.69410759865549E-16 0.349087221077984 -> xyz=-0.0491247882 0.2246558260 0 rpy=0 1.5707963267949 1.5707963267949
- joint Right_Shoulder_X: axis 1 0 0 -> 0 0 1; origin xyz=-0.167642819137822 0.257434208389716 -0.0153204612848374 rpy=5.79452944416604E-17 -1.59192802633449E-16 -0.349087221077984 -> xyz=-0.167642819137822 -0.257434208389716 0.0153204612848374 rpy=-1.5707963267949 0 -1.221709106
- joint Right_Shoulder_Y: origin xyz=0 0 0 rpy=0 0 9.22447382158831E-33 -> xyz=0 0 0 rpy=1.5707963267949 -1.221709106 0
- joint Right_Wrist_X: axis 1 0 0 -> 0 0 1; origin xyz=0 0 0 rpy=0 0 0 -> xyz=0 0 0 rpy=0 -1.5707963267949 1.5707963267949
- joint Right_Wrist_Y: origin xyz=0 0 0 rpy=0 0 0 -> xyz=0 0 0 rpy=0 -1.5707963267949 1.5707963267949
- joint Right_Wrist_Z: axis 0 -1 0 -> 0 0 1; origin xyz=0 -0.209559555159009 0.000544952004672944 rpy=0 0 0 -> xyz=0 0.209559555159009 0 rpy=-1.5707963267949 0 0
